File: Board Files/Motherboard.kicad_pcb (KiCad board)
At the start: 2 copper layers, 106.1 x 155 mm, 84 parts, among them P1 72-Pin Connector, P2 PowerSw, P3 ResetSw, P4 Controller_Port, P6 RF-Mod, Q1 2SA937, Q2 2SC2021, T1 08RB01, U1 6116 (WRAM), U2 74HC373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

Commit message: + Migrate to Kicad 9 + Fix symbol issues caused by Kicad 6+ library and symbol name changes + Change "HEX BUFFERS" label to "CONTROLLER HEX BUFFERS" to match OpenTendo + Migrate legacy symbol .lib to Kicad 6+ .kicad_sym format + Fix incorrect "thermal relief" setting on zone, changed to correct "solid" + Updated ignored DRC tests to better match the board design
Connections:
- net /CPU-R~W renamed /CPU-R~{W}
- net /PPU-~A13 renamed /PPU-~{A13}
- net /PPU-~CE renamed /PPU-~{CE}
- net /PPU-~RD renamed /PPU-~{RD}
- net /PPU-~WE renamed /PPU-~{WE}
- net /VRAM-~CE renamed /VRAM-~{CE}
- net /WRAM-~CE renamed /WRAM-~{CE}
- net /~IRQ renamed /~{IRQ}
- net /~NMI renamed /~{NMI}
- net /~OE1 renamed /~{OE1}
- net /~OE2 renamed /~{OE2}
- net /~ROMSEL renamed /~{ROMSEL}
- net /~RST renamed /~{RST}
Other:
- net class Default removed
- net class Thin removed
